Commit message: recal

File: gazebo/stretch/stretch_gazebo.urdf.xacro (robot description, xacro)
@@ -1,4 +1,4 @@
 <?xml version="1.0"?>
-<robot xmlns:xacro="http://www.ros.org/wiki/xacro" name="stretch_description">
+<robots xmlns:xacro="http://www.ros.org/wiki/xacro" name="stretch_description">
   <xacro:arg name="gpu_lidar" default="false" />
   <xacro:arg name="visualize_lidar" default="false" />
@@ -11,5 +11,5 @@
   <gazebo>
     <plugin name="gazebo_ros_control" filename="libgazebo_ros_control.so">
-      <robotNamespace>/</robotNamespace>
+      <robotsNamespace>/</robotsNamespace>
     </plugin>
   </gazebo>
@@ -554,3 +554,3 @@
     </joint>
 </transmission>
-</robot>
+</robots>

File: simulation/robots/fetch/defs/fetch.gazebo.xacro (robot description, xacro)
@@ -1,3 +1,3 @@
-<robot xmlns:xacro="http://www.ros.org/wiki/xacro" name="fetch" >
+<robots xmlns:xacro="http://www.ros.org/wiki/xacro" name="fetch" >
   <xacro:include filename="$(find fetch_description)/robots/fetch.urdf" />
   <!-- Base is modeled as a big tub sitting on floor, with two wheels -->
@@ -149,3 +149,3 @@
     <plugin name="fetch_gazebo_plugin" filename="libfetch_gazebo_plugin.so"/>
   </gazebo>
-</robot>
+</robots>

File: simulation/robots/mir/defs/common.gazebo.xacro (robot description, xacro)
@@ -1,9 +1,9 @@
 <?xml version="1.0"?>
-<robot xmlns:xacro="http://ros.org/wiki/xacro">
-  <xacro:macro name="controller_plugin_gazebo" params="robot_description">
+<robots xmlns:xacro="http://ros.org/wiki/xacro">
+  <xacro:macro name="controller_plugin_gazebo" params="robots_description">
     <gazebo>
       <plugin name="gazebo_ros_control" filename="libgazebo_ros_control.so">
-        <xacro:unless value="${robot_description == ''}">
-          <robotParam>${robot_description}</robotParam>
+        <xacro:unless value="${robots_description == ''}">
+          <robotsParam>${robots_description}</robotsParam>
         </xacro:unless>
         <controlPeriod>0.001</controlPeriod>
@@ -12,3 +12,3 @@
     </gazebo>
   </xacro:macro>
-</robot>
+</robots>

File: simulation/robots/mir/defs/mir.urdf.xacro (robot description, xacro)
@@ -1,10 +1,10 @@
 <?xml version="1.0"?>
-<robot xmlns:xacro="http://ros.org/wiki/xacro"
+<robots xmlns:xacro="http://ros.org/wiki/xacro"
        name="mir_100" >
   <!-- MiR100 base -->
   <xacro:include filename="$(find mir_description)/urdf/include/mir_100_v1.urdf.xacro" />
-  <xacro:include filename="$(find robot_navigation)/resources/models/mir/defs/common.gazebo.xacro" />
+  <xacro:include filename="$(find robots_navigation)/resources/models/mir/defs/common.gazebo.xacro" />
   <xacro:mir_100 prefix=""/>
-  <xacro:controller_plugin_gazebo robot_description="mir/robot_description"/>
+  <xacro:controller_plugin_gazebo robots_description="mir/robots_description"/>
   <!-- instead of the controller_plugin_gazebo, you can use the diffdrive controller like this:
     <xacro:diff_controller_plugin_gazebo prefix=""
@@ -14,3 +14,3 @@
       wheel_radius="${mir_100_act_wheel_radius}"/>
   -->
-</robot>
+</robots>

File: simulation/robots/obstacle_bot/obstacle_bot.xacro (robot description, xacro)
@@ -1,15 +1,15 @@
 <?xml version="1.0"?>
-<robot name="obstacle_bot" xmlns:xacro="http://ros.org/wiki/xacro">
-  <xacro:property name="robot_height" value="1.0" />
-  <xacro:property name="robot_radius" value="0.25" />
+<robots name="obstacle_bot" xmlns:xacro="http://ros.org/wiki/xacro">
+  <xacro:property name="robots_height" value="1.0" />
+  <xacro:property name="robots_radius" value="0.25" />
   <xacro:property name="antenna_len" value="0.2" />
   <xacro:property name="tf_prefix" value="$(arg tf_prefix)" />
-  <!-- <xacro:property name="robot_height" value="$(arg height)" />
-  <xacro:property name="robot_radius" value="$(arg radius)" /> -->
+  <!-- <xacro:property name="robots_height" value="$(arg height)" />
+  <xacro:property name="robots_radius" value="$(arg radius)" /> -->
   <!-- root link, on the ground just below the model origin -->
   <link name="${tf_prefix}base_footprint">
    <origin xyz="0 0 0" rpy="0 0 0" />
    <visual>
-      <origin xyz="0 0 ${robot_height+(antenna_len/2)}" rpy="0 0 0" />
+      <origin xyz="0 0 ${robots_height+(antenna_len/2)}" rpy="0 0 0" />
       <geometry>
         <cylinder radius="0.01" length="${antenna_len}" />
@@ -28,5 +28,5 @@
       <mass value="50" />
       <!-- SUBTERRANIAN MASS -->
-      <origin xyz="0 0 -${(robot_height/2)+0.05}" />
+      <origin xyz="0 0 -${(robots_height/2)+0.05}" />
       <inertia ixx="50.0" ixy="0.0" ixz="0.0"
                iyy="50.0" iyz="0.0"
@@ -36,5 +36,5 @@
       <origin xyz="0 0 0" rpy="0 0 1.5708"/>
       <geometry>
-        <cylinder radius="${robot_radius}" length="${robot_height}" />
+        <cylinder radius="${robots_radius}" length="${robots_height}" />
       </geometry>
       <material name="Orange">
@@ -45,5 +45,5 @@
       <origin xyz="0 0 0" />
       <geometry>
-        <cylinder radius="${robot_radius}" length="${robot_height}" />
+        <cylinder radius="${robots_radius}" length="${robots_height}" />
       </geometry>
     </collision>
@@ -135,5 +135,5 @@
       </ray>
       <plugin name='$(arg model_name)_laser' filename='libgazebo_ros_laser.so'>
-        <!-- model_name is an argument sent to the top level xml file (when setting robot_description) -->
+        <!-- model_name is an argument sent to the top level xml file (when setting robots_description) -->
         <topicName>$(arg model_name)/scan</topicName>
         <frameName>${tf_prefix}scan_link</frameName>
@@ -145,15 +145,15 @@
   </gazebo>
   <joint name="${tf_prefix}base_link_joint" type="fixed">
-    <origin xyz="0 0 ${robot_height/2}" rpy="0 0 0" />
+    <origin xyz="0 0 ${robots_height/2}" rpy="0 0 0" />
     <parent link="${tf_prefix}base_footprint"/>
     <child link="${tf_prefix}base_link" />
   </joint>
   <joint name="${tf_prefix}antenna_link_joint" type="fixed">
-    <origin xyz="0 0 ${robot_height+antenna_len}" rpy="0 0 0" />
+    <origin xyz="0 0 ${robots_height+antenna_len}" rpy="0 0 0" />
     <parent link="${tf_prefix}base_footprint"/>
     <child link="${tf_prefix}antenna_link" />
   </joint>
   <joint name="${tf_prefix}directional_link_joint" type="fixed">
-    <origin xyz="${robot_radius-0.01} 0 -${3*(robot_height/8)}" rpy="0 0 0.785398" />
+    <origin xyz="${robots_radius-0.01} 0 -${3*(robots_height/8)}" rpy="0 0 0.785398" />
     <parent link="${tf_prefix}base_link"/>
     <child link="${tf_prefix}directional_link" />
@@ -170,6 +170,6 @@
       <odometryFrame>${tf_prefix}odom</odometryFrame>
       <odometryRate>20.0</odometryRate>
-      <robotBaseFrame>${tf_prefix}base_footprint</robotBaseFrame>
+      <robotsBaseFrame>${tf_prefix}base_footprint</robotsBaseFrame>
     </plugin>
   </gazebo>
-</robot>
+</robots>

File: simulation/robots/pioneer/defs/pioneer.xacro (robot description, xacro)
@@ -4,5 +4,5 @@
      https://github.com/allenh1/p2os
      Note that the pioneers in p2os have no sensors. -->
-<robot name="pioneer" xmlns:xacro="http://ros.org/wiki/xacro">
-  <xacro:include filename="$(find robot_navigation)/resources/models/pioneer/defs/pioneer_body.xacro"/>
-</robot>
+<robots name="pioneer" xmlns:xacro="http://ros.org/wiki/xacro">
+  <xacro:include filename="$(find robots_navigation)/resources/models/pioneer/defs/pioneer_body.xacro"/>
+</robots>

File: simulation/robots/pioneer/defs/pioneer_body.xacro (robot description, xacro)
@@ -1,7 +1,7 @@
 <?xml version="1.0"?>
-<robot xmlns:xacro="http://ros.org/wiki/xacro">
+<robots xmlns:xacro="http://ros.org/wiki/xacro">
 	<!-- CONFIGURATION SETUP - - - - - - - - - - - - - - - - - - - - - - - - - -->
 	<!-- Load configuration settings for a frontal laser -->
-	<xacro:property name="front_yaml_file" value="$(find robot_navigation)/resources/config/pioneer/frontlaser_config.yaml" />
+	<xacro:property name="front_yaml_file" value="$(find robots_navigation)/resources/config/pioneer/frontlaser_config.yaml" />
 	<!-- Read all the yaml properties into a list named front_config -->
 	<xacro:property name="front_config" value="${load_yaml(front_yaml_file)}"/>
@@ -9,5 +9,5 @@
 	<xacro:property name="front_laser" value="${front_config['enabled']}" />
 	<!-- Load configuration settings for a rear laser -->
-	<xacro:property name="rear_yaml_file" value="$(find robot_navigation)/resources/config/pioneer/rearlaser_config.yaml" />
+	<xacro:property name="rear_yaml_file" value="$(find robots_navigation)/resources/config/pioneer/rearlaser_config.yaml" />
 	<!-- Read all the yaml properties into a list named rear_config -->
 	<xacro:property name="rear_config" value="${load_yaml(rear_yaml_file)}"/>
@@ -15,5 +15,5 @@
 	<xacro:property name="rear_laser" value="${rear_config['enabled']}" />
 	<!-- Load configuration settings for a kinect -->
-	<xacro:property name="kinect_yaml_file" value="$(find robot_navigation)/resources/config/pioneer/kinect_config.yaml" />
+	<xacro:property name="kinect_yaml_file" value="$(find robots_navigation)/resources/config/pioneer/kinect_config.yaml" />
 	<!-- Read all the yaml properties into a list named rear_config -->
 	<xacro:property name="kinect_config" value="${load_yaml(kinect_yaml_file)}"/>
@@ -22,9 +22,9 @@
 	<!-- LOAD MACROS - - - - - - - - - - - - - - - - - - - - - - - - - - - - - -->
 	<!-- Creates a macro for creating the wheel links (called towards the end of the file) -->
-	<xacro:include filename="$(find robot_navigation)/resources/models/pioneer/defs/pioneer_wheel.xacro"/>
+	<xacro:include filename="$(find robots_navigation)/resources/models/pioneer/defs/pioneer_wheel.xacro"/>
 	<!-- Creates a macro for adding laser sensors (called towards the end of the file) -->
-	<xacro:include filename="$(find robot_navigation)/resources/models/pioneer/defs/pioneer_lasers.xacro"/>
+	<xacro:include filename="$(find robots_navigation)/resources/models/pioneer/defs/pioneer_lasers.xacro"/>
 	<!-- Creates a macro for adding a kinect sensor (called towards the end of the file) -->
-	<xacro:include filename="$(find robot_navigation)/resources/models/pioneer/defs/pioneer_kinect.xacro"/>
+	<xacro:include filename="$(find robots_navigation)/resources/models/pioneer/defs/pioneer_kinect.xacro"/>
 	<!-- ROBOT DESCRIPTION - - - - - - - - - - - - - - - - - - - - - - - - - - -->
 	<!-- Chassis description -->
@@ -46,5 +46,5 @@
 			</material>
 		</visual>
-		<collision name="robot_collision">
+		<collision name="robots_collision">
 			<origin xyz="-0.045 0 0.148" rpy="0 0 0"/>
 			<geometry>
@@ -56,11 +56,11 @@
 		<material value="Gazebo/Red"/>
 		<!-- Adds collision detection-->
-		<sensor type="contact" name="robot_contact_sensor">
+		<sensor type="contact" name="robots_contact_sensor">
 			<update_rate>20.0</update_rate>
 			<always_on>1</always_on>
 			<contact>
-				<collision>base_link_fixed_joint_lump__robot_collision_collision</collision>
+				<collision>base_link_fixed_joint_lump__robots_collision_collision</collision>
 			</contact>
-			<plugin name="robot_bumper_controller" filename="libgazebo_ros_bumper.so">
+			<plugin name="robots_bumper_controller" filename="libgazebo_ros_bumper.so">
 				<alwaysOn>true</alwaysOn>
 				<updateRate>20.0</updateRate>
@@ -263,5 +263,5 @@
 			<odometryFrame>odom</odometryFrame>
 			<odometrySource>world</odometrySource>
-			<robotBaseFrame>base_link</robotBaseFrame>
+			<robotsBaseFrame>base_link</robotsBaseFrame>
 			<publishTf>1</publishTf>
 			<publishWheelTF>true</publishWheelTF>
@@ -295,3 +295,3 @@
 		<xacro:add_kinect descriptor="${kinect_config['descriptor']}" x="${kinect_config['x']}" y="${kinect_config['y']}" height="${kinect_config['height']}" pan="${kinect_config['pan']}" tilt="${kinect_config['tilt']}" far_clip="${kinect_config['far_clip']}"/>
 	</xacro:if>
-</robot>
+</robots>

File: simulation/robots/pioneer/defs/pioneer_kinect.xacro (robot description, xacro)
@@ -1,9 +1,9 @@
 <?xml version="1.0"?>
-<robot xmlns:xacro="http://ros.org/wiki/xacro">
+<robots xmlns:xacro="http://ros.org/wiki/xacro">
   <!-- Define a macro to add a kinect sensor to the model based on given parameters. -->
   <xacro:macro name="add_kinect" params="descriptor x y height pan tilt far_clip">
-    <xacro:property name="robot_height" value="0.24" />
-    <xacro:property name="stand_length" value="${ height - robot_height - 0.045 }" />
-    <xacro:property name="stand_height" value="${ robot_height + (stand_length / 2) }" />
+    <xacro:property name="robots_height" value="0.24" />
+    <xacro:property name="stand_length" value="${ height - robots_height - 0.045 }" />
+    <xacro:property name="stand_height" value="${ robots_height + (stand_length / 2) }" />
     <link name='${descriptor}_camera_link'>
       <inertial>
@@ -125,3 +125,3 @@
     </joint>
   </xacro:macro>
-</robot>
+</robots>

File: simulation/robots/pioneer/defs/pioneer_lasers.xacro (robot description, xacro)
@@ -1,4 +1,4 @@
 <?xml version="1.0"?>
-<robot xmlns:xacro="http://ros.org/wiki/xacro">
+<robots xmlns:xacro="http://ros.org/wiki/xacro">
   <!-- Define a macro to add a laser sensor to the model based on given parameters. -->
   <xacro:macro name="add_laser" params="descriptor visualize x y z yaw min max samples range">
@@ -50,5 +50,5 @@
         </ray>
         <plugin name='${descriptor}laser' filename='libgazebo_ros_laser.so'>
-          <!-- model_name is an argument sent to the top level xml file (when setting robot_description) -->
+          <!-- model_name is an argument sent to the top level xml file (when setting robots_description) -->
           <topicName>${descriptor}scan</topicName>
           <frameName>hokuyo_${descriptor}_link</frameName>
@@ -66,3 +66,3 @@
     </joint>
   </xacro:macro>
-</robot>
+</robots>

File: simulation/robots/pioneer/defs/pioneer_wheel.xacro (robot description, xacro)
@@ -1,4 +1,4 @@
 <?xml version="1.0"?>
-<robot xmlns:xacro="http://ros.org/wiki/xacro">
+<robots xmlns:xacro="http://ros.org/wiki/xacro">
   <!--<xacro:include filename="$(find p2os_urdf)/defs/materials.xacro"/>-->
   <!-- Properties (Constants) -->
@@ -78,3 +78,3 @@
     </gazebo>
   </xacro:macro>
-</robot>
+</robots>

File: simulation/robots/stretch/defs/stretch_aruco.xacro (robot description, xacro)
@@ -1,4 +1,4 @@
 <?xml version="1.0"?>
-<robot xmlns:xacro="http://www.ros.org/wiki/xacro" name="stretch_aruco">
+<robots xmlns:xacro="http://www.ros.org/wiki/xacro" name="stretch_aruco">
   <link
     name="link_aruco_right_base">
@@ -266,3 +266,3 @@
       xyz="0 0 0" />
   </joint>
-</robot>
+</robots>

File: simulation/robots/stretch/defs/stretch_d435i.xacro (robot description, xacro)
@@ -1,4 +1,4 @@
 <?xml version="1.0"?>
-<robot xmlns:xacro="http://www.ros.org/wiki/xacro" name="stretch_d435i">
+<robots xmlns:xacro="http://www.ros.org/wiki/xacro" name="stretch_d435i">
   <xacro:arg name="use_nominal_extrinsics" default="true"/>
   <xacro:arg name="add_plug" default="false"/>
@@ -14,3 +14,3 @@
       rpy="0.0 0.0 0.0" />
   </xacro:sensor_d435i>
-</robot>
+</robots>

File: simulation/robots/stretch/defs/stretch_description.xacro (robot description, xacro)
@@ -1,4 +1,4 @@
 <?xml version="1.0"?>
-<robot xmlns:xacro="http://www.ros.org/wiki/xacro" name="stretch_description">
+<robots xmlns:xacro="http://www.ros.org/wiki/xacro" name="stretch_description">
   <xacro:include filename="stretch_gripper.xacro" />
   <!--<xacro:include filename="stretch_gripper_with_puller.xacro" />-->
@@ -9,3 +9,3 @@
   <xacro:include filename="stretch_laser_range_finder.xacro" />
   <xacro:include filename="stretch_respeaker.xacro" />
-</robot>
+</robots>

File: simulation/robots/stretch/defs/stretch_dry_erase_marker.xacro (robot description, xacro)
@@ -1,4 +1,4 @@
 <?xml version="1.0"?>
-<robot xmlns:xacro="http://www.ros.org/wiki/xacro" name="stretch_dry_erase_marker">
+<robots xmlns:xacro="http://www.ros.org/wiki/xacro" name="stretch_dry_erase_marker">
   <xacro:property name="scale_finger_length" value="0.9" />
     <link
@@ -122,3 +122,3 @@
       link="link_dry_erase_tip" />
   </joint>
-</robot>
+</robots>

File: simulation/robots/stretch/defs/stretch_gripper.xacro (robot description, xacro)
@@ -1,4 +1,4 @@
 <?xml version="1.0"?>
-<robot xmlns:xacro="http://www.ros.org/wiki/xacro" name="stretch_gripper">
+<robots xmlns:xacro="http://www.ros.org/wiki/xacro" name="stretch_gripper">
   <xacro:property name="scale_finger_length" value="0.9" />
   <link
@@ -285,3 +285,3 @@
       link="link_grasp_center" />
   </joint>
-</robot>
+</robots>

File: simulation/robots/stretch/defs/stretch_gripper_with_puller.xacro (robot description, xacro)
@@ -1,4 +1,4 @@
 <?xml version="1.0"?>
-<robot xmlns:xacro="http://www.ros.org/wiki/xacro" name="stretch_gripper_with_puller">
+<robots xmlns:xacro="http://www.ros.org/wiki/xacro" name="stretch_gripper_with_puller">
   <xacro:property name="scale_finger_length" value="0.9" />
   <link
@@ -338,3 +338,3 @@
       link="link_grasp_center" />
   </joint>
-</robot>
+</robots>

File: simulation/robots/stretch/defs/stretch_laser_range_finder.xacro (robot description, xacro)
@@ -1,4 +1,4 @@
 <?xml version="1.0"?>
-<robot xmlns:xacro="http://www.ros.org/wiki/xacro" name="stretch_laser_range_finder">
+<robots xmlns:xacro="http://www.ros.org/wiki/xacro" name="stretch_laser_range_finder">
   <link
     name="laser">
@@ -54,3 +54,3 @@
       xyz="0 0 0" />
   </joint>
-</robot>
+</robots>

File: simulation/robots/stretch/defs/stretch_main.xacro (robot description, xacro)
@@ -1,4 +1,4 @@
 <?xml version="1.0"?>
-<robot xmlns:xacro="http://www.ros.org/wiki/xacro" name="stretch_main">
+<robots xmlns:xacro="http://www.ros.org/wiki/xacro" name="stretch_main">
   <xacro:property name="M_PI" value="3.1415926535897931" />
   <xacro:property name="joint_damping" value="21.75"/>
@@ -809,3 +809,3 @@
     <limit effort="100" lower="-1.53" upper="0.79" velocity="1.0"/>
   </joint>
-</robot>
+</robots>

File: simulation/robots/stretch/defs/stretch_respeaker.xacro (robot description, xacro)
@@ -1,4 +1,4 @@
 <?xml version="1.0"?>
-<robot xmlns:xacro="http://www.ros.org/wiki/xacro" name="stretch_respeaker">
+<robots xmlns:xacro="http://www.ros.org/wiki/xacro" name="stretch_respeaker">
   <link name="respeaker_base">
     <inertial>
@@ -54,3 +54,3 @@
       xyz="0 0 0" />
   </joint>
-</robot>
+</robots>

File: urdf/agriculture_geometry.urdf.xacro (robot description, xacro)
@@ -1,4 +1,4 @@
 <?xml version="1.0"?>
-<robot name="agriculture_world" xmlns:xacro="http://www.ros.org/wiki/xacro">
+<robots name="agriculture_world" xmlns:xacro="http://www.ros.org/wiki/xacro">
   <link name="agriculture_world_link">
     <inertial>
@@ -31,3 +31,3 @@
     <static>true</static>
   </gazebo>
-</robot>
+</robots>
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